Commit message: Update URDF configuration in src

File: src/my_robot_arm_pkg/urdf/urdf_moveit.urdf (robot description, URDF)
Before this commit: robot urdf_moveit, 10 links, 9 joints
Joints:
- joint J3: limit lower=- upper=3.14 effort=0.92 velocity=6.16 -> lower=-0.1 upper=3.14 effort=0.92 velocity=6.16

Commit message: Add src and uros_ws updates: bridge_node, moveit configs, and micro-ROS workspace

File: src/my_robot_arm_pkg/urdf/urdf_moveit.urdf (robot description, URDF)
Before this commit: robot urdf_moveit, 10 links, 9 joints
Joints:
- joint J1: limit lower=0 upper=3.14 effort=0.92 velocity=6.16 -> lower=-0.1 upper=3.14 effort=0.92 velocity=6.16
- joint J4: limit lower=0 upper=3.14 effort=0.13 velocity=8.72 -> lower=-0.1 upper=3.14 effort=0.13 velocity=8.72
